File: gamegirl.kicad_pcb (KiCad board)
At the start: 2 copper layers, 58 parts, among them J1 Conn_01x07_Socket, J2 Conn_01x14_Socket, J3 Conn_01x04_Socket, SW1 EN, SW10 select, SW12 SS12D07VG4 087, SW2 up, SW3 down, SW4 left, SW5 right, SW6 A, SW7 B, SW8 BOOT, SW9 start, U1 ESP32-WROOM-32, U2 AP2112K-3.3, U3 CH340N_C2977777

Commit message: why is this display so big
Parts:
- C1, C2, C4, D1, D2, R3, R4, R6, U2, U3: moved to B.Cu
- moved R4 69.5 mm to (178.0, 45.5), turned to 180 degrees
- moved R3 67.9 mm to (180.5, 48.8), turned to 180 degrees
- moved J3 65.8 mm to (230.8, 67.2)
- moved SW12 62.2 mm to (213.2, 51.5)
- moved U2 55.6 mm to (174.2, 41.0), turned to 180 degrees
- moved C3 54.2 mm to (167.2, 38.8)
- moved C4 53.0 mm to (163.2, 38.8), turned to 180 degrees
- moved R6 52.7 mm to (100.9, 44.0), turned to -90 degrees
- moved C1 49.4 mm to (168.8, 42.0)
- moved C2 47.2 mm to (163.1, 42.0)
- moved SW10 32.0 mm to (180.0, 58.8)
- moved SW5 21.1 mm to (96.2, 65.8)
- moved U3 20.7 mm to (173.8, 49.5), turned to -90 degrees
- moved SW1 17.9 mm to (167.8, 63.5), turned to 0 degrees
- moved J2 7.16 mm to (108.2, 52.5)
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Routing:
- net /tx: track 0.00 -> 47.2 mm, vias 0 -> 2
- net /rx: track 0.00 -> 42.5 mm, vias 0 -> 2
- net VBUS: track 0.00 -> 20.8 mm
- net +3V3: track 0.00 -> 17.7 mm, vias 0 -> 1
- net GND: track 0.00 -> 11.6 mm, vias 0 -> 12
- net usb dm: track 0.00 -> 10.5 mm
- net usb dp: track 0.00 -> 9.88 mm
- net Net-(U3-UD-): track 0.00 -> 6.73 mm
- net Net-(U1-EN): track 0.00 -> 4.55 mm
- net Net-(U3-UD+): track 0.00 -> 3.64 mm
Other:
- board outline added: 186.8 x 65 mm

Commit message: rough layout
Parts:
- C3, R17, R5, SW12: moved to B.Cu
- moved H6 119.8 mm to (87.6, 107.1)
- moved H5 115.9 mm to (86.4, 56.9)
- moved C10 106.9 mm to (54.6, 154.6)
- moved C9 106.9 mm to (54.6, 151.6)
- moved R11 106.9 mm to (59.0, 160.6)
- moved R15 106.9 mm to (63.4, 160.6)
- moved R2 106.9 mm to (50.2, 160.6)
- moved R7 106.9 mm to (54.6, 160.6)
- moved C13 106.9 mm to (59.1, 148.6)
- moved R1 106.9 mm to (50.2, 157.6)
- moved R12 106.9 mm to (59.0, 163.5)
- moved R13 106.9 mm to (59.0, 166.4)
- moved R14 106.9 mm to (63.4, 157.6)
- moved R16 106.9 mm to (63.4, 163.5)
- moved R8 106.9 mm to (54.6, 163.5)
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Connections:
- J2 pad 1: unconnected-(J2-Pin_1-Pad1) -> +3V3
- J2 pad 10: /GPIO2 -> unconnected-(J2-Pin_10-Pad10)
- J2 pad 11: /GPIO4 -> unconnected-(J2-Pin_11-Pad11)
- J2 pad 12: /GPIO5 -> unconnected-(J2-Pin_12-Pad12)
- J2 pad 13: GND -> unconnected-(J2-Pin_13-Pad13)
- J2 pad 14: +3V3 -> unconnected-(J2-Pin_14-Pad14)
- J2 pad 2: unconnected-(J2-Pin_2-Pad2) -> GND
- J2 pad 3: unconnected-(J2-Pin_3-Pad3) -> /GPIO5
- J2 pad 4: unconnected-(J2-Pin_4-Pad4) -> /GPIO4
- J2 pad 5: unconnected-(J2-Pin_5-Pad5) -> /GPIO2
- J2 pad 6: /GPIO19 -> /GPIO23
- J2 pad 7: /LCD_BRIGHT -> /GPIO18
- J2 pad 8: /GPIO18 -> /LCD_BRIGHT
- J2 pad 9: /GPIO23 -> /GPIO19
Routing:
- net VBUS: track 20.8 -> 123.3 mm, vias 0 -> 1
- net /GPIO22: track 0.00 -> 85.7 mm, vias 0 -> 1
- net /GPIO25: track 0.00 -> 61.5 mm, vias 0 -> 1
- net /GPIO26: track 0.00 -> 60.6 mm, vias 0 -> 1
- net +3V3: track 17.7 -> 58.7 mm, vias 1 -> 2
- net /tx: track 47.2 -> 11.9 mm, vias 2 -> 0
- net /rx: track 42.5 -> 12.1 mm, vias 2 -> 0
- net Net-(U1-EN): track 4.55 -> 19.9 mm
- net /GAIN: track 0.00 -> 8.61 mm
- net GND: track 11.6 -> 16.7 mm
- net usb dm: track 10.5 -> 15.6 mm
- net Net-(D1-A): track 0.00 -> 3.46 mm
- net Net-(U3-UD+): track 3.64 -> 5.17 mm
- net usb dp: track 9.88 -> 8.60 mm
- net Net-(U3-UD-): track 6.73 -> 7.33 mm
Other:
- board size 186.8 x 65 mm -> 175 x 70 mm

Commit message: more progress
Parts:
- C10, C11, C12, C13, C5, C6, C7, C8, C9, R1, R10, R11, R12, R14, R15, R2, R7, R8: moved to B.Cu
- D2: moved to F.Cu
- moved R12 203.0 mm to (242.0, 75.8), turned to 180 degrees
- moved R11 199.8 mm to (238.0, 71.8), turned to 180 degrees
- moved C10 193.9 mm to (237.8, 91.0), turned to 180 degrees
- moved C9 193.7 mm to (231.8, 73.2), turned to 180 degrees
- moved C13 192.0 mm to (224.8, 51.5)
- moved R14 188.7 mm to (242.0, 96.8), turned to 180 degrees
- moved R15 168.5 mm to (222.8, 105.8), turned to 180 degrees
- moved R2 121.5 mm to (118.8, 60.2), turned to 180 degrees
- moved R1 119.1 mm to (123.2, 63.5), turned to 180 degrees
- moved R13 117.4 mm to (128.8, 72.0), turned to 90 degrees
- moved R16 104.4 mm to (82.9, 61.0), turned to -90 degrees
- moved R7 101.2 mm to (96.1, 68.2), turned to 180 degrees
- moved R9 89.2 mm to (84.8, 82.5)
- moved R8 70.3 mm to (86.8, 101.0)
- moved SW1 31.7 mm to (186.7, 60.1)
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Routing:
- net +3V3: track 58.7 -> 86.3 mm, vias 2 -> 4
- net VBUS: track 123.3 -> 130.9 mm
- net Net-(D1-A): track 3.46 -> 0.00 mm
- net /GAIN: track 8.61 -> 11.6 mm

Commit message: disasterous layout
Parts:
- R13, R9: moved to B.Cu
- moved D2 151.7 mm to (233.9, 66.5), turned to 180 degrees
- moved R16 145.6 mm to (228.4, 66.8), turned to 0 degrees
- moved R6 48.6 mm to (95.8, 104.6), turned to 0 degrees
- moved BOOT 16.7 mm to (155.5, 76.8)
- moved R13 10.2 mm to (138.2, 68.2), turned to 180 degrees
- moved R14 9.72 mm to (232.8, 93.8), turned to 0 degrees
- moved SW1 8.64 mm to (178.5, 57.2)
- moved R7 2.77 mm to (93.5, 67.2)
- moved R1 1.55 mm to (122.0, 62.6), turned to 90 degrees
- moved R2 0.65 mm to (118.2, 60.7), turned to -90 degrees
- turned C11 to 0 degrees
- turned R9 to 180 degrees
- renumbered SW8 to BOOT
Routing:
- net /left: track 0.00 -> 101.0 mm, vias 0 -> 2
- net /status: track 0.00 -> 91.6 mm, vias 0 -> 3
- net /select: track 0.00 -> 88.1 mm, vias 0 -> 1
- net /down: track 0.00 -> 86.4 mm, vias 0 -> 3
- net /start: track 0.00 -> 83.1 mm
- net /right: track 0.00 -> 73.2 mm, vias 0 -> 2
- net /GPIO15: track 0.00 -> 72.7 mm, vias 0 -> 1
- net /GPIO19: track 0.00 -> 63.3 mm, vias 0 -> 1
- net /GPIO14: track 0.00 -> 61.4 mm, vias 0 -> 1
- net /GPIO23: track 0.00 -> 61.1 mm, vias 0 -> 1
- net /GPIO12: track 0.00 -> 58.6 mm, vias 0 -> 1
- net /GPIO18: track 0.00 -> 58.3 mm, vias 0 -> 1
- net /GPIO13: track 0.00 -> 57.2 mm
- net /up: track 0.00 -> 45.2 mm
- net /GPIO4: track 0.00 -> 45.0 mm, vias 0 -> 1
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Other:
- board text added: "GAMEGIRL™"

Commit message: traces of doom and despair
Parts:
- SW12: moved to F.Cu
- moved SW12 218.6 mm to (17.0, 8.75), turned to -90 degrees
- moved J1 200.8 mm to (25.2, 3.17)
- moved D2 108.6 mm to (140.2, 11.5)
- moved R16 108.6 mm to (134.7, 11.8)
- moved SW7 106.8 mm to (143.5, 23.8)
- moved H8 104.9 mm to (120.2, 57.2)
- moved SW9 104.2 mm to (143.5, 42.0)
- moved J3 103.1 mm to (120.2, 31.4)
- moved C10 100.4 mm to (145.4, 51.7)
- moved C11 100.4 mm to (138.8, 69.5)
- moved C12 100.4 mm to (130.7, 59.8)
- moved R15 100.4 mm to (130.3, 66.4)
- moved H4 99.5 mm to (153.5, 64.0)
- moved H7 99.4 mm to (120.2, 13.2)
- moved SW6 99.4 mm to (131.5, 31.0)
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Routing:
- net VBUS: track 130.9 -> 21.0 mm, vias 1 -> 0
- net /left: track 101.0 -> 10.3 mm, vias 2 -> 0
- net /select: track 88.1 -> 0.00 mm, vias 1 -> 0
- net /GPIO22: track 85.7 -> 0.00 mm, vias 1 -> 0
- net /down: track 86.4 -> 2.21 mm, vias 3 -> 0
- net /status: track 91.6 -> 7.45 mm, vias 3 -> 1
- net /start: track 83.1 -> 0.00 mm
- net /GPIO26: track 60.6 -> 0.00 mm, vias 1 -> 0
- net /GPIO25: track 61.5 -> 2.41 mm
- net /right: track 73.2 -> 23.2 mm, vias 2 -> 1
- net /up: track 45.2 -> 1.99 mm
- net /GPIO14: track 61.4 -> 35.1 mm
- net /GPIO15: track 72.7 -> 49.0 mm
- net GND: track 59.6 -> 36.2 mm
- net /GPIO12: track 58.6 -> 37.9 mm
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Other:
- board size 175 x 70 mm -> 160 x 70 mm

Commit message: final? layout
Parts:
- D2: footprint LED_SMD:LED_0603_1608Metric -> LED_THT:LED_D3.0mm
- moved C5 119.6 mm to (84.8, 114.2), turned to 90 degrees
- moved R7 116.9 mm to (81.2, 117.0), turned to 90 degrees
- moved R10 114.9 mm to (86.5, 122.5), turned to 180 degrees
- moved C8 111.3 mm to (77.0, 125.8), turned to -90 degrees
- moved R9 110.5 mm to (65.0, 119.5), turned to 90 degrees
- moved R14 108.3 mm to (199.0, 142.5), turned to 180 degrees
- moved C6 105.8 mm to (71.5, 131.5)
- moved C13 105.3 mm to (84.0, 94.5), turned to -90 degrees
- moved BOOT 104.8 mm to (143.2, 113.8)
- moved C1 104.8 mm to (120.8, 92.5)
- moved C4 104.8 mm to (151.2, 93.2)
- moved D1 104.8 mm to (94.3, 93.5)
- moved H1 104.8 mm to (59.2, 96.2)
- moved H2 104.8 mm to (60.0, 153.5)
- moved H3 104.8 mm to (206.8, 96.5)
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Routing:
- net +3V3: track 116.1 -> 440.0 mm, vias 5 -> 8
- net GND: track 36.2 -> 345.2 mm, vias 12 -> 9
- net /down: track 2.21 -> 104.8 mm, vias 0 -> 1
- net /GPIO26: track 0.00 -> 102.3 mm, vias 0 -> 1
- net /left: track 10.3 -> 110.8 mm, vias 0 -> 2
- net /GPIO25: track 2.41 -> 100.1 mm, vias 1 -> 2
- net /up: track 1.99 -> 97.6 mm, vias 0 -> 2
- net /select: track 0.00 -> 92.3 mm, vias 0 -> 1
- net /start: track 0.00 -> 84.8 mm, vias 0 -> 1
- net /right: track 23.2 -> 102.6 mm
- net /B: track 0.00 -> 76.0 mm, vias 0 -> 1
- net /A: track 0.00 -> 64.0 mm, vias 0 -> 1
- net /GPIO22: track 0.00 -> 56.4 mm, vias 0 -> 1
- net /status: track 7.45 -> 59.1 mm
- net VBUS: track 21.0 -> 69.6 mm, vias 0 -> 2
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- added copper zone on F.Cu, net GND

Commit message: final?
Parts:
- removed R6: RK09K1130AP5, easyeda2kicad:RES-ADJ-TH_RK09K1130AJ3
- moved R16 0.35 mm to (184.0, 99.0)
- renumbered SW10 to SELECT, SW9 to START, BOOT to SW8, SW2 to up
Connections:
- J2 pad 8: /LCD_BRIGHT -> +3V3
- J3 pad 3: /GPIO12 -> /GPIO17
- U1 pad 14: /GPIO12 -> unconnected-(U1-IO12-Pad14)
- U1 pad 28: unconnected-(U1-IO17-Pad28) -> /GPIO17
Routing:
- net /GPIO17: track 0.00 -> 53.7 mm, vias 0 -> 1
- net /GPIO12: track 37.9 -> 0.00 mm, vias 1 -> 0
- net /LCD_BRIGHT: track 26.2 -> 0.00 mm
- net GND: track 345.2 -> 321.7 mm
- net +3V3: track 440.0 -> 442.3 mm, vias 8 -> 9
- net /GPIO14: track 35.1 -> 33.0 mm
Other:
- board size 160 x 70 mm -> 160 x 70.2 mm
- board text added: "404 Display not found"
- board text added: "Made by: Samridh Prabhakar Sabastian Hamilton Aadithya Vasudevan Mahdi El Husseini Michael Wu Wilbert Chu"
- board text added: "this better work"
- board text added: "vol"

Commit message: final gerber files
Parts:
- removed U3: CH340N_C2977777, easyeda2kicad:SOP-8_L4.9-W3.9-P1.27-LS6.0-BL
- added Q1: MUN5211DW1, Package_TO_SOT_SMD:SOT-363_SC-70-6, B.Cu at (124.8, 107.2)
- added R18: 10k, Resistor_SMD:R_0805_2012Metric, B.Cu at (173.5, 135.6)
- added R6: 10k, Resistor_SMD:R_0805_2012Metric, B.Cu at (97.0, 115.0)
- added U4: CH340C, Package_SO:SOIC-16_3.9x9.9mm_P1.27mm, B.Cu at (119.0, 106.3)
- D1: value LED -> PWR
- D2: value LED -> STATUS
- R16: moved to B.Cu
- R3, R4: footprint Resistor_SMD:R_0805_2012Metric -> Resistor_SMD:R_0603_1608Metric
- moved R13 6.01 mm to (128.0, 114.0)
- moved R4 2.38 mm to (112.5, 107.5)
- moved R3 1.52 mm to (113.0, 103.5)
- moved C3 1.47 mm to (154.5, 95.5), turned to 0 degrees
- renumbered SELECT to SW10, up to SW2
Connections:
- net Net-(U1-EN) renamed /en
- net Net-(U1-IO0) renamed /boot
- J2 pad 8: +3V3 -> unconnected-(J2-Pin_8-Pad8)
- USB1 pad : (no net) -> GND
Routing:
- net /en: track 33.9 -> 63.6 mm, vias 0 -> 2
- net GND: track 321.7 -> 297.2 mm, vias 9 -> 10
- net +3V3: track 442.3 -> 460.4 mm, vias 9 -> 11
- net Net-(Q1A-E1): track 0.00 -> 16.7 mm, vias 0 -> 2
- net Net-(Q1A-B1): track 0.00 -> 11.2 mm
- net /GPIO15: track 49.0 -> 54.3 mm
- net /GPIO5: track 43.6 -> 48.6 mm, vias 1 -> 2
- net Net-(U4-UD+): track 5.17 -> 9.57 mm
- net /boot: track 23.0 -> 24.6 mm
- net usb dm: track 15.6 -> 14.2 mm
- net Net-(U4-UD-): track 7.33 -> 8.45 mm
- net /tx: track 11.9 -> 12.8 mm
- net /GPIO22: track 56.4 -> 57.2 mm
- net /GPIO4: track 45.0 -> 44.5 mm
- net /GPIO13: track 38.8 -> 38.2 mm
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