File: gamegirl.kicad_sch (KiCad schematic)
At the start: 58 parts, among them J1 Conn_01x07_Socket, J2 Conn_01x14_Socket, J3 Conn_01x04_Socket, SW1 EN, SW10 select, SW12 SS12D07VG4 087, SW2 up, SW3 down, SW4 left, SW5 right, SW6 A, SW7 B, SW8 BOOT, SW9 start, U1 ESP32-WROOM-32, U2 AP2112K-3.3, U3 CH340N_C2977777

Commit message: final? layout
Connections:
- net +3V3: now also J2.1 (Pin_1); no longer J2.14 (Pin_14)
- net GND: now also J2.2 (Pin_2); no longer J2.13 (Pin_13)
- net GPIO18: now also J2.7 (Pin_7); no longer J2.8 (Pin_8)
- net GPIO19: now also J2.9 (Pin_9); no longer J2.6 (Pin_6)
- net GPIO2: now also J2.5 (Pin_5); no longer J2.10 (Pin_10)
- net GPIO23: now also J2.6 (Pin_6); no longer J2.9 (Pin_9)
- net GPIO4: now also J2.4 (Pin_4); no longer J2.11 (Pin_11)
- net GPIO5: now also J2.3 (Pin_3); no longer J2.12 (Pin_12)
- net LCD_BRIGHT: now also J2.8 (Pin_8); no longer J2.7 (Pin_7)
Changed lines of the file:
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@@
 	(text "CS"
 		(exclude_from_sim no)
-		(at 195.072 140.97 0)
+		(at 195.072 118.364 0)
 		(effects
 			(font
@@
 	(text "SCK"
 		(exclude_from_sim no)
-		(at 195.326 131.064 0)
+		(at 195.834 128.778 0)
 		(effects
 			(font
@@
 	(text "MISO"
 		(exclude_from_sim no)
-		(at 195.834 125.984 0)
+		(at 195.58 133.35 0)
 		(effects
 			(font
@@
 	(text "DC"
 		(exclude_from_sim no)
-		(at 195.072 136.398 0)
+		(at 195.58 123.444 0)
 		(effects
 			(font
@@
 	(text "MOSI"
 		(exclude_from_sim no)
-		(at 195.834 133.604 0)
+		(at 196.088 125.984 0)
 		(effects
 			(font
@@
 	(text "RST"
 		(exclude_from_sim no)
-		(at 195.326 138.684 0)
+		(at 195.326 121.158 0)
 		(effects
 			(font
@@
 	)
 	(no_connect
+		(at 187.96 135.89)
+	)
+	(no_connect
 		(at 77.47 77.47)
 	)
@@
 	)
 	(no_connect
-		(at 187.96 115.57)
-	)
-	(no_connect
-		(at 187.96 118.11)
-	)
-	(no_connect
 		(at 77.47 72.39)
 	)
 	(no_connect
-		(at 187.96 123.19)
-	)
-	(no_connect
 		(at 130.81 162.56)
 	)
 	(no_connect
-		(at 187.96 113.03)
+		(at 187.96 143.51)
 	)
 	(no_connect
@@
 	)
 	(no_connect
-		(at 219.71 101.6)
+		(at 187.96 138.43)
 	)
 	(no_connect
-		(at 187.96 120.65)
+		(at 219.71 101.6)
 	)
 	(no_connect
@@
 	)
 	(no_connect
+		(at 187.96 140.97)
+	)
+	(no_connect
+		(at 187.96 146.05)
+	)
+	(no_connect
 		(at 247.65 34.29)
 	)
@@
 	(wire
 		(pts
+			(xy 181.61 115.57) (xy 187.96 115.57)
+		)
+		(stroke
+			(width 0)
+			(type default)
+		)
+	)
+	(wire
+		(pts
 			(xy 60.96 175.26) (xy 60.96 177.8)
 		)
@@
 	)
 	(label "GPIO23"
-		(at 187.96 133.35 180)
+		(at 187.96 125.73 180)
 		(effects
 			(font
@@
 	)
 	(label "GPIO19"
-		(at 187.96 125.73 180)
+		(at 187.96 133.35 180)
 		(effects
 			(font
@@
 	)
 	(label "GPIO5"
-		(at 187.96 140.97 180)
+		(at 187.96 118.11 180)
 		(effects
 			(font
@@
 	)
 	(label "GPIO2"
-		(at 187.96 135.89 180)
+		(at 187.96 123.19 180)
 		(effects
 			(font
@@
 	)
 	(label "LCD_BRIGHT"
-		(at 187.96 128.27 180)
+		(at 187.96 130.81 180)
 		(effects
 			(font
@@
 	)
 	(label "GPIO4"
-		(at 187.96 138.43 180)
+		(at 187.96 120.65 180)
 		(effects
 			(font
@@
 	)
 	(label "GPIO18"
-		(at 187.96 130.81 180)
+		(at 187.96 128.27 180)
 		(effects
 			(font
@@
 	(symbol
 		(lib_id "power:+3V3")
-		(at 187.96 146.05 180)
+		(at 187.96 113.03 0)
 		(unit 1)
 		(body_style 1)
@@
 		(in_pos_files yes)
 		(dnp no)
-		(fields_autoplaced yes)
 		(property "Reference" "#PWR019"
-			(at 187.96 142.24 0)
+			(at 187.96 116.84 0)
 			(hide yes)
 			(show_name no)
@@
 		)
 		(property "Value" "+3V3"
-			(at 187.96 151.13 0)
+			(at 181.356 110.49 0)
 			(show_name no)
 			(do_not_autoplace no)
@@
 					(size 1.27 1.27)
 				)
+				(justify left)
 			)
 		)
 		(property "Footprint" ""
-			(at 187.96 146.05 0)
+			(at 187.96 113.03 0)
 			(hide yes)
 			(show_name no)
@@
 		)
 		(property "Datasheet" ""
-			(at 187.96 146.05 0)
+			(at 187.96 113.03 0)
 			(hide yes)
 			(show_name no)
@@
 		)
 		(property "Description" "Power symbol creates a global label with name \"+3V3\""
-			(at 187.96 146.05 0)
+			(at 187.96 113.03 0)
 			(hide yes)
 			(show_name no)
@@
 		(dnp no)
 		(property "Reference" "J2"
-			(at 193.802 113.284 0)
+			(at 194.818 147.828 0)
 			(show_name no)
 			(do_not_autoplace no)
@@
 		)
 		(property "Value" "Conn_01x14_Socket"
-			(at 193.802 115.824 0)
+			(at 194.818 150.368 0)
 			(show_name no)
 			(do_not_autoplace no)
@@
 	(symbol
 		(lib_id "power:GND")
-		(at 187.96 143.51 270)
+		(at 181.61 115.57 180)
 		(unit 1)
 		(body_style 1)
@@
 		(fields_autoplaced yes)
 		(property "Reference" "#PWR018"
-			(at 181.61 143.51 0)
+			(at 181.61 109.22 0)
 			(hide yes)
 			(show_name no)
@@
 		)
 		(property "Value" "GND"
-			(at 184.15 143.5099 90)
+			(at 184.15 114.2999 0)
 			(show_name no)
 			(do_not_autoplace no)
@@
 		)
 		(property "Footprint" ""
-			(at 187.96 143.51 0)
+			(at 181.61 115.57 0)
 			(hide yes)
 			(show_name no)
@@
 		)
 		(property "Datasheet" ""
-			(at 187.96 143.51 0)
+			(at 181.61 115.57 0)
 			(hide yes)
 			(show_name no)
@@
 		)
 		(property "Description" "Power symbol creates a global label with name \"GND\" , ground"
-			(at 187.96 143.51 0)
+			(at 181.61 115.57 0)
 			(hide yes)
 			(show_name no)

Commit message: final?
Parts:
- removed R6: RK09K1130AP5, easyeda2kicad:RES-ADJ-TH_RK09K1130AJ3, symbol easyeda2kicad:RK09K1130AP5
Connections:
- net LCD_BRIGHT is gone; now on net +3V3: J2.8 (Pin_8)
- net GPIO17: now reaches U1.28 (IO17)
- net GPIO17: now also J3.3 (Pin_3)
- net GPIO12: no longer names the net of U1.14 (IO12)
- net GPIO12: no longer J3.3 (Pin_3)
Other:
- note added: "LED"

Commit message: final gerber files
Parts:
- removed U3: CH340N_C2977777, easyeda2kicad:SOP-8_L4.9-W3.9-P1.27-LS6.0-BL, symbol easyeda2kicad:CH340N_C2977777
- added Q1: MUN5211DW1, Package_TO_SOT_SMD:SOT-363_SC-70-6, symbol Transistor_BJT:MUN5211DW1
- added R18, R6: 10k, Resistor_SMD:R_0805_2012Metric, symbol Device:R_Small_US
- added U4: CH340C, Package_SO:SOIC-16_3.9x9.9mm_P1.27mm, symbol Interface_USB:CH340C
- R3, R4: footprint Resistor_SMD:R_0805_2012Metric -> Resistor_SMD:R_0603_1608Metric
Connections:
- net +3V3: now also R18.2, R6.2, U4.16 (VCC), U4.4 (V3); no longer J2.8 (Pin_8)
- net GND: now also U4.1 (GND)
- net GPIO15: now also R18.1
- net GPIO5: now also R6.1
- net rx: now also U4.3 (RXD)
- net tx: now also U4.2 (TXD)
- net boot: now reaches R13.1, SW8.1, U1.25 (IO0)
- net boot: now also Q1.6 (C1)
- net en: now reaches C2.1, R5.1, SW1.2, U1.3 (EN)
- net en: now also Q1.3 (C2)
- net at R3.2: now also U4.5 (UD+)
- net at R4.2: now also U4.6 (UD-)
- new net: Q1.1 (E1), Q1.5 (B2), U4.13 (~{DTR})
- new net: Q1.2 (B1), Q1.4 (E2), U4.14 (~{RTS})
- no-connect marks 16 -> 19
Other:
- note added: "CS protection resistors"
- moved on the sheet: J2, J3, R3, R4
